File: sata-backplane.kicad_pcb (KiCad board)
At the start: 4 copper layers, 56 x 43 mm, 11 parts, among them J1 SATA_POWER_15, J10 SATA_1, J11 SATA_COMBINED_1, J20 SATA_2, J21 SATA_COMBINED_2

Commit message: Update PCB with final touch
Parts:
- removed kibuzzard-63A87A6D (x2): G***, kibuzzard-63A87A6D
- removed kibuzzard-63A87AA0 (x2): G***, kibuzzard-63A87AA0
- removed kibuzzard-63A87D87: G***, kibuzzard-63A87D87
- removed kibuzzard-63A9DCD5: G***, kibuzzard-63A9DCD5
- added REF**: OSHW-Logo_5.7x6mm_SilkScreen, Symbol:OSHW-Logo_5.7x6mm_SilkScreen, F.Cu at (73.1, 41.5)
- added kibuzzard-63B1B127: G***, kibuzzard-63B1B127, F.Cu at (37.3, 54.8)
- added kibuzzard-63B1B175: G***, kibuzzard-63B1B175, F.Cu at (63.3, 35.6)
- added kibuzzard-63B1B175: G***, kibuzzard-63B1B175, B.Cu at (56.5, 28.6)
- added kibuzzard-63B1B17B: G***, kibuzzard-63B1B17B, F.Cu at (63.3, 47.3)
- added kibuzzard-63B1B17B: G***, kibuzzard-63B1B17B, B.Cu at (56.5, 54.4)
- added kibuzzard-63B1B180: G***, kibuzzard-63B1B180, F.Cu at (37.2, 45.9)
Other:
- board text added: "JLCJLCJLCJLC"
- board text added: "V1.0 CC BY-SA"
- board text removed: "GPL v3"
- board text removed: "V1.0"

Commit message: Update connectors with V1.0 experience
Parts:
- removed REF**: OSHW-Logo_5.7x6mm_SilkScreen, Symbol:OSHW-Logo_5.7x6mm_SilkScreen
Other:
- board text added: "V1.1 CC BY-SA"
- board text removed: "V1.0 CC BY-SA"
